File: PCBs/Pneumatactors_1Xiao_CompactControl/Pneumatactors_1Xiao_CompactControl.kicad_pcb (KiCad board)
At the start: 2 copper layers, 25 x 55 mm, 20 parts, among them J1 Valve_1, J2 Valve_2, J3 Pump, J4 Pogo Connection, Q1 IRLML2060, Q2 IRLML2060, U1 SeeeduinoXIAO, U2 Pololu 2990, U3 TS01AQE

Commit message: 2025-03-27 00:00:06
Other:
- board text added: "P-1"
- board text added: "V-1"
- board text added: "V-2"
Changed lines of the file:
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@@
     (effects (font (size 1 1) (thickness 0.15)) (justify left bottom mirror))
+  )
+  (gr_text "V-1" (at 22.225 12.065) (layer "F.SilkS")
+    (effects (font (size 1 1) (thickness 0.15)))
+  )
+  (gr_text "P-1" (at 22.225 30.48) (layer "F.SilkS")
+    (effects (font (size 1 1) (thickness 0.15)))
+  )
+  (gr_text "V-2" (at 22.225 20.955) (layer "F.SilkS")
+    (effects (font (size 1 1) (thickness 0.15)))
   )
   (dimension (type aligned) (layer "Dwgs.User")
